File: EDA/TrailCurrentBorealis/TrailCurrentBorealis.kicad_pcb (KiCad board)
At the start: 2 copper layers, 68.5 x 49.1 mm, 11 parts, among them IC1 SN65HVD230DR, J2 S4B-XH-SM4-TB, U1 ESP32-S3-Zero, U2 GY-SGP30, U3 Mini560, U4 SHT31-D-TempHumidity

Commit message: Revised version of the case design. Grbls added for mfg
Parts:
- added LOGO: TrailCurrentLogo_Text, TrailCurrentFootprints:TrailCurrentLogo_Text, F.Cu at (123.5, 92.1)
- added LOGO: TrailCurrentLogo_Icon, TrailCurrentFootprints:TrailCurrentLogo_Icon, B.Cu at (135.9, 91.5)
Connections:
- U1 pad 12: (no net) -> unconnected-(U1-GPIO9-Pad12)
- U1 pad 13: (no net) -> unconnected-(U1-GPIO10-Pad13)
- U1 pad 14: (no net) -> unconnected-(U1-GPIO11-Pad14)
- U1 pad 17: (no net) -> unconnected-(U1-RX-Pad17)
- U1 pad 18: (no net) -> unconnected-(U1-TX-Pad18)
- U1 pad 19: (no net) -> unconnected-(U1-GPIO45-Pad19)
- U1 pad 20: (no net) -> unconnected-(U1-GPIO42-Pad20)
- U1 pad 21: (no net) -> unconnected-(U1-GPIO41-Pad21)
- U1 pad 22: (no net) -> unconnected-(U1-GPIO40-Pad22)
- U1 pad 23: (no net) -> unconnected-(U1-GPIO39-Pad23)
- U1 pad 24: (no net) -> unconnected-(U1-GPIO38-Pad24)
- U1 pad 25: (no net) -> unconnected-(U1-GPIO18-Pad25)
- U1 pad 26: (no net) -> unconnected-(U1-GPIO17-Pad26)
- U1 pad 4: (no net) -> unconnected-(U1-GPIO1-Pad4)
- U1 pad 6: (no net) -> unconnected-(U1-GPIO3-Pad6)
- U1 pad 7: (no net) -> unconnected-(U1-GPIO4-Pad7)
Routing:
- net +3.3V: track 111.8 -> 11.2 mm
- net GND: track 83.0 -> 18.9 mm, vias 1 -> 4
- net +5V: track 74.3 -> 71.7 mm
- net +12V: track 51.0 -> 48.5 mm
- net SCL: track 61.7 -> 63.0 mm
- net SDA: track 74.6 -> 75.6 mm
- added copper zone on F.Cu, net +3.3V
Other:
- board text added: "Borealis v1.0.0"
- board text added: "TrailCurrent"

Commit message: WIP EDA advancing the PCB further with better buck converter and reverse polarity protection
Parts:
- removed U3: Mini560, TrailCurrentFootprints:Mini560
- added C1: 10uF, Capacitor_SMD:C_1206_3216Metric_Pad1.33x1.80mm_HandSolder, F.Cu at (138.4, 119.6)
- added C2: 22uF, Capacitor_SMD:C_1206_3216Metric_Pad1.33x1.80mm_HandSolder, F.Cu at (131.7, 115.8)
- added C3: 22uF, Capacitor_SMD:C_1206_3216Metric_Pad1.33x1.80mm_HandSolder, F.Cu at (131.7, 113.4)
- added C4: 100nF, Capacitor_SMD:C_1206_3216Metric_Pad1.33x1.80mm_HandSolder, F.Cu at (137.8, 110.7)
- added D2: SS34, TrailCurrentFootprints:SS34, F.Cu at (181.9, 107.6)
- added D3: SMBJ24CA-13-F, TrailCurrentFootprints:SMBJ24CA-13-F, F.Cu at (180.5, 112.9)
- added FB1: BLM31PG121SN1L, TrailCurrentFootprints:BLM31PG121SN1L, F.Cu at (185.4, 110.9)
- added FB2: BLM31PG121SN1L, TrailCurrentFootprints:BLM31PG121SN1L, F.Cu at (178.3, 108.3)
- added IC2: AP63205QWU-7, TrailCurrentFootprints:AP63205QWU7, F.Cu at (137.0, 114.5)
- added L1: 0420CDMCCDS-4R7MC, TrailCurrentFootprints:0420CDMCCDS-4R7MC, F.Cu at (132.9, 119.6)
- moved LOGO 11.6 mm to (131.3, 102.1)
Connections:
- J2 pad 1: +12V -> /+12V_RAW
- U1 pad 5: DHT_READING -> unconnected-(U1-GPIO2-Pad5)
Routing:
- net +5V: track 71.7 -> 108.1 mm
- net +12V: track 48.5 -> 15.1 mm
- net /+12V_RAW: track 0.00 -> 23.7 mm
- net GND: track 18.9 -> 33.3 mm, vias 4 -> 7
- net Net-(IC2-SW): track 0.00 -> 10.8 mm
- net Net-(IC2-BST): track 0.00 -> 7.16 mm
- net Net-(D2-K): track 0.00 -> 3.44 mm
- net Net-(D3-Pad1): track 0.00 -> 3.14 mm
